Commit message: Fix three real bugs blocking native KUKA grasp generation
- assets/kuka/kuka.urdf: kuka_joint8 was missing the KUKA Y-gripper's real
  180deg-about-Z flange mount rotation (present in the hardware-canonical
  gripper_mount_joint and in fabrica_kuka.urdf's kuka_hand_joint, but dropped
  when this arm-only IK-chain URDF was ported). Restored it and corrected the
  now-stale "no mount rotation" comments in kuka.urdf and geometry.py's
  get_kuka_basis_directions(). Needed for real-hardware/Isaac-Gym joint-angle
  consistency (the render_motion_plan.py planning/rendering path itself is
  algebraically invariant to this rotation via util_arm.py's rest-pose
  self-calibration, so it wasn't the cause of any visible render artifact).

- assets/kuka/{visual,collision}/*.obj (22 files): every KUKA mesh (hand,
  both fingers, all 8 arm links) was baked in meters while the rest of the
  codebase -- Panda meshes, part meshes, all cm-based grasp-offset math --
  uses centimeters, a 100x scale mismatch. Rescaled all vertices by 100x.
  This was the actual blocker for KUKA grasp generation: finger meshes 100x
  too small at a correctly-positioned (cm-scale) grasp pose never overlapped
  the part mesh, so contact-point detection silently returned zero points
  for ~96% of candidates.

- planning/run_grasp_arm_gen.py: applied the finger-mesh face-normal winding
  flip to 'kuka' (previously only 'panda'), per the TODO already left in that
  function -- confirmed via the same contact-point diagnostic that KUKA's
  independently-converted finger meshes need it too.

- utils/parallel.py: parallel_worker now catches exceptions from the wrapped
  worker instead of dying silently. An uncaught exception in one of the 50
  parallel IK workers (e.g. scipy's `x0 is infeasible` on a bad initial
  guess -- a separate, pre-existing edge case, not caused by the above)
  never pushed a result to the queue, so parallel_execute's final drain loop
  blocked forever waiting on that one dead worker instead of just treating
  the candidate as failed like every other rejection path already does.

Net effect verified via a full plumbers_block --arm kuka --gripper kuka
run_planning.sh pass: no hang, and grasp-candidate contact-point detection
now works instead of failing near-100% of the time. Grasp generation still
comes back empty for this specific assembly because of a separate,
pre-existing, already-documented gap -- planning/robot/workcell.py's KUKA
board-mount position is a placeholder copied from Panda's layout ("pending
real reach-based tuning"), causing near-universal gripper-ground collisions
-- left unfixed since correcting it needs real reach/mounting data, not a
guess.

Co-Authored-By: Claude Sonnet 5 <noreply@anthropic.com>

File: assets/kuka/kuka.urdf (robot description, URDF)
Before this commit: robot kuka, 9 links, 8 joints
Joints:
- joint kuka_joint8: origin xyz=0 0 0.0308 rpy=0 0 0 -> xyz=0 0 0.0308 rpy=0 0 3.14159265
